Commit message: Update robot_core.xacro

File: description/robot_core.xacro (robot description, xacro)
@@ -0,0 +1,31 @@
+<?xml version="1.0"?>
+<robot xmlns:xacro="http://www.ros.org/wiki/xacro" >
+   <material name="white">
+    <color rgba="1 1 1 1"/>
+  </material>
+  <material name="orange">
+    <color rgba="1 0.5 0 1"/>
+  </material>
+  <material name="blue">
+    <color rgba="0.2 0.2 1 1"/>
+  </material>
+  <material name="black">
+    <color rgba="0 0 0 1"/>
+  </material>
+<link name="base_link">
+</link>
+<joint name="chassis_joint" type="fixed">
+     <parent link="base_link"/>
+     <child link="chassis"/>
+     <origin xyz="-0.1 0 0"/>
+</joint>
+<link name="chassis">
+     <visual>
+          <origin xyz="0.15 0 0.075"
+          <geometry>
+                <box size="0.3 0.3 0.15"/>
+          </geometry>
+          <material name="white"/>
+     </visual>
+</link>
+</robot>

Commit message: Update robot_core.xacro

File: description/robot_core.xacro (robot description, xacro)
@@ -22,5 +22,5 @@
 <link name="chassis">
      <visual>
-          <origin xyz="0.15 0 0.075"
+          <origin xyz="0.15 0 0.075"/>
           <geometry>
                 <box size="0.3 0.3 0.15"/>

Commit message: Update robot_core.xacro

File: description/robot_core.xacro (robot description, xacro)
@@ -22,7 +22,7 @@
 <link name="chassis">
      <visual>
-          <origin xyz="0.15 0 0.075"/>
+          <origin xyz="0.15 0 0.15"/>
           <geometry>
-                <box size="0.3 0.3 0.15"/>
+                <box size="0.3 0.3 0.3"/>
           </geometry>
           <material name="white"/>

Commit message: Update robot_core.xacro

File: description/robot_core.xacro (robot description, xacro)
@@ -13,6 +13,8 @@
     <color rgba="0 0 0 1"/>
   </material>
+      <!-- BASE LINK --!>
 <link name="base_link">
 </link>
+     <!-- CHASSIS LINK --!>
 <joint name="chassis_joint" type="fixed">
      <parent link="base_link"/>
@@ -22,10 +24,40 @@
 <link name="chassis">
      <visual>
-          <origin xyz="0.15 0 0.15"/>
+          <origin xyz="0.15 0 0.075"
           <geometry>
-                <box size="0.3 0.3 0.3"/>
+                <box size="0.3 0.3 0.15"/>
           </geometry>
           <material name="white"/>
      </visual>
 </link>
+    <!-- LEFT WHEEL LINK --!>
+<joint name="left_wheel_joint" type="continous">
+     <parent link="base_link"/>
+     <child link="left wheel"/>
+     <origin xyz="0 0.175 0" rpy="-${pi/2} 0 0"/>
+     <axis xyz="0 0 1"/>
+</joint>
+<link name="left_wheel">
+     <visual>
+          <geometry>
+                <cycliner radius="0.05" length="0.04"/>
+          </geometry>
+          <material name="blue"/>
+     </visual>
+</link>
+<!-- RIGHT WHEEL LINK --!>
+<joint name="right_wheel_joint" type="continous">
+     <parent link="base_link"/>
+     <child link="rigwheel"/>
+     <origin xyz="0 -0.175 0" rpy="${pi/2} 0 0"/>
+     <axis xyz="0 0 -1"/>
+</joint>
+<link name="right_wheel">
+     <visual>
+          <geometry>
+                <cycliner radius="0.05" length="0.04"/>
+          </geometry>
+          <material name="blue"/>
+     </visual>
+</link>
 </robot>
